File: PushBuzz/PushBuzz.kicad_sch (KiCad schematic)
At the start: 12 parts, among them J2 nRF52840 Dongle, Q1 BSH105, Q2 BSH105, Q3 BSH105, Q4 BSH105, Q5 DMP31D0U, SW1 12x12x? SMD Pushbutton

Commit message: Add alternate references
Parts:
- J1: value (none) -> 282834-6; footprint (none) -> TerminalBlock_TE-Connectivity:TerminalBlock_TE_282834-6_1x06_P2.54mm_Horizontal
Other:
- note added: "Alt: DMG3414U"
- note added: "Alt: Si2301CDS"
Changed lines of the file:
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@@
     (stroke (width 0) (type default) (color 0 0 0 0))
+  )
+  (text "Alt: DMG3414U" (at 165.735 61.595 0)
+    (effects (font (size 1.27 1.27)) (justify left bottom))
+  )
+  (text "Alt: DMG3414U" (at 87.63 87.63 0)
+    (effects (font (size 1.27 1.27)) (justify left bottom))
+  )
+  (text "Alt: Si2301CDS" (at 172.085 37.465 0)
+    (effects (font (size 1.27 1.27)) (justify left bottom))
+  )
+  (text "Alt: DMG3414U" (at 124.46 61.595 0)
+    (effects (font (size 1.27 1.27)) (justify left bottom))
+  )
+  (text "Alt: DMG3414U" (at 124.46 87.63 0)
+    (effects (font (size 1.27 1.27)) (justify left bottom))
   )
   (text "BAT+\nBAT-\nLED+\nLED-\nPB\nPB" (at 58.42 70.485 180)
@@
     (in_bom yes) (on_board yes) (fields_autoplaced)
     (property "Reference" "J1" (id 0) (at 60.96 50.8 0))
-    (property "Value" "" (id 1) (at 60.96 53.34 0))
-    (property "Footprint" "" (id 2) (at 60.96 62.23 0)
+    (property "Value" "282834-6" (id 1) (at 60.96 53.34 0))
+    (property "Footprint" "TerminalBlock_TE-Connectivity:TerminalBlock_TE_282834-6_1x06_P2.54mm_Horizontal" (id 2) (at 60.96 62.23 0)
       (effects (font (size 1.27 1.27)) hide)
     )
